Commit message: update to noetic devel

File: src/scorpio/scorpio_description/urdf/_d435.urdf.xacro (robot description, xacro)
@@ -46,5 +46,5 @@
         <geometry>
           <!-- <box size="${d435_cam_width} ${d435_cam_height} ${d435_cam_depth}"/> -->
-          <mesh filename="package://scorpio_description/meshes/d435.dae" />
+          <mesh filename="package://spark_description/meshes/spark/sensors/spark_d435.dae" />
           <!--mesh filename="$(find realsense2_description)/meshes/d435.dae" /-->
         </geometry>
@@ -117,3 +117,6 @@
     <link name="camera_color_optical_frame"/>
   </xacro:macro>
+  <xacro:sensor_d435 parent="base_link">
+	<origin xyz="0.16 0 0.229500" rpy="0 0 0"/>
+  </xacro:sensor_d435>
 </robot>

File: src/scorpio/scorpio_description/urdf/scorpio_silver.urdf.xacro (robot description, xacro)
@@ -8,8 +8,5 @@
   	<xacro:include filename="$(find scorpio_description)/urdf/base/car_base_silver.urdf"/>
 	<xacro:include filename="$(find ydlidar_g2)/urdf/ydlidar.urdf" />
-	<xacro:include filename="$(find scorpio_description)/urdf/_d435.urdf.xacro" />
-	<sensor_d435 parent="base_link">
-		<origin xyz="0.16 0 0.229500" rpy="0 0 0"/>
-	</sensor_d435>
+	<xacro:include filename="$(find scorpio_description)/urdf/sensors/_d435.urdf.xacro"/>
 	<!--xacro:include filename="$(find scorpio_description)/urdf/sensors/scorpio_camera.urdf"/-->
 </robot>
